File: X-10A42V-DDSB-PSU-DUAL-IN-ONE-10A-42V-SYMMETRICAL-PSU-FOR-POWER-AMP.kicad_pcb (KiCad board)
At the start: 2 copper layers, 214.3 x 85.7 mm, 72 parts, among them K101 SLA-24VDC-SL-A

Commit message: Update
Parts:
- added C207: 470uF, CUSTOM-FOOTPRINTS:CP_Radial_D10.0mm_P5.00mm, F.Cu at (187.3, 225.7)
- added C208: 470uF, CUSTOM-FOOTPRINTS:CP_Radial_D10.0mm_P5.00mm, F.Cu at (219.1, 225.7)
- added C209: 470uF, CUSTOM-FOOTPRINTS:CP_Radial_D10.0mm_P5.00mm, F.Cu at (161.9, 198.8)
- added C210: 470uF, CUSTOM-FOOTPRINTS:CP_Radial_D10.0mm_P5.00mm, F.Cu at (244.5, 198.8)
- added C211: 470uF, CUSTOM-FOOTPRINTS:CP_Radial_D10.0mm_P5.00mm, F.Cu at (203.2, 198.8)
- added CNT101: 2376582-2, CUSTOM-FOOTPRINTS:PCB_TAB_250_FASTON_TPBR, F.Cu at (112.7, 201.9)
- added CNT102: 2376582-2, CUSTOM-FOOTPRINTS:PCB_TAB_250_FASTON_TPBR, F.Cu at (68.6, 201.9)
- added CNT103: 2376582-2, CUSTOM-FOOTPRINTS:PCB_TAB_250_FASTON_TPBR, F.Cu at (112.7, 226.7)
- added CNT104: 2376582-2, CUSTOM-FOOTPRINTS:PCB_TAB_250_FASTON_TPBR, F.Cu at (68.3, 226.7)
- added CNT105: 2376582-2, CUSTOM-FOOTPRINTS:PCB_TAB_250_FASTON_TPBR, F.Cu at (90.5, 194.9)
- added CNT213: 22-27-2031, CUSTOM-FOOTPRINTS:Molex_KK-254_AE-6410-03A_1x03_P2.54mm_Vertical, F.Cu at (159.4, 225.7)
- added CNT214: 22-27-2021, CUSTOM-FOOTPRINTS:Molex_KK-254_AE-6410-02A_1x02_P2.54mm_Vertical, F.Cu at (133.3, 203.8)
- added CNT215: 22-27-2021, CUSTOM-FOOTPRINTS:Molex_KK-254_AE-6410-02A_1x02_P2.54mm_Vertical, F.Cu at (273.1, 206.4)
- added CNT216: 22-27-2041, CUSTOM-FOOTPRINTS:Molex_KK-254_AE-6410-04A_1x04_P2.54mm_Vertical, F.Cu at (133.3, 212.4)
- added CNT217: 22-27-2041, CUSTOM-FOOTPRINTS:Molex_KK-254_AE-6410-04A_1x04_P2.54mm_Vertical, F.Cu at (273.1, 220.0)
- added D203: VS-2KBP005, CUSTOM-FOOTPRINTS:Diode_Bridge_Vishay_KBPM, F.Cu at (197.4, 225.8)
- added FB202: Ferrite Bead, Ferrite_THT:LairdTech_28C0236-0JW-10, F.Cu at (170.5, 225.7)
- added J101: PF0002-28, CUSTOM-FOOTPRINTS:BULGIN-IEC-Connector-PF0002-28, B.Cu at (90.5, 214.6)
- added REF**: DRILL_1.27mm, CUSTOM-FOOTPRINTS:DRILL_1.27mm, F.Cu at (118.7, 226.1)
- added REF**: DRILL_1.27mm, CUSTOM-FOOTPRINTS:DRILL_1.27mm, F.Cu at (268.6, 191.5)
- added REF**: DRILL_1.27mm, CUSTOM-FOOTPRINTS:DRILL_1.27mm, F.Cu at (95.2, 191.5)
- added REF**: DRILL_1.27mm_11.43mm, CUSTOM-FOOTPRINTS:DRILL_1.27mm_11.43mm, F.Cu at (118.7, 209.9)
- added REF**: DRILL_1.27mm, CUSTOM-FOOTPRINTS:DRILL_1.27mm, F.Cu at (245.1, 191.5)
- added REF**: DRILL_1.27mm, CUSTOM-FOOTPRINTS:DRILL_1.27mm, F.Cu at (270.8, 191.5)
- added REF**: DRILL_1.27mm, CUSTOM-FOOTPRINTS:DRILL_1.27mm, F.Cu at (221.6, 191.5)
- added REF**: Hole_2.7mm, CUSTOM-FOOTPRINTS:Hole_2.7mm, F.Cu at (133.0, 196.8)
- added REF**: DRILL_1.27mm, CUSTOM-FOOTPRINTS:DRILL_1.27mm, F.Cu at (118.7, 198.1)
- added REF**: DRILL_1.27mm, CUSTOM-FOOTPRINTS:DRILL_1.27mm, F.Cu at (65.1, 191.5)
- added REF**: DRILL_1.27mm, CUSTOM-FOOTPRINTS:DRILL_1.27mm, F.Cu at (226.1, 191.5)
- added REF**: DRILL_1.27mm, CUSTOM-FOOTPRINTS:DRILL_1.27mm, F.Cu at (204.8, 191.5)
- added REF**: DRILL_1.27mm, CUSTOM-FOOTPRINTS:DRILL_1.27mm, F.Cu at (127.6, 221.6)
- added REF**: DRILL_1.27mm, CUSTOM-FOOTPRINTS:DRILL_1.27mm, F.Cu at (118.7, 200.3)
- added REF**: DRILL_1.27mm, CUSTOM-FOOTPRINTS:DRILL_1.27mm, F.Cu at (118.7, 191.5)
- added REF**: DRILL_1.27mm_11.43mm, CUSTOM-FOOTPRINTS:DRILL_1.27mm_11.43mm, F.Cu at (190.8, 191.5)
- added REF**: Hole_2.7mm, CUSTOM-FOOTPRINTS:Hole_2.7mm, F.Cu at (273.4, 196.8)
- added REF**: DRILL_1.27mm, CUSTOM-FOOTPRINTS:DRILL_1.27mm, F.Cu at (254.0, 191.5)
- added REF**: DRILL_1.27mm, CUSTOM-FOOTPRINTS:DRILL_1.27mm, F.Cu at (118.7, 217.2)
- added REF**: DRILL_1.27mm, CUSTOM-FOOTPRINTS:DRILL_1.27mm, F.Cu at (123.2, 191.5)
- added REF**: DRILL_1.27mm, CUSTOM-FOOTPRINTS:DRILL_1.27mm, F.Cu at (127.6, 230.5)
- added REF**: DRILL_1.27mm, CUSTOM-FOOTPRINTS:DRILL_1.27mm, F.Cu at (78.4, 191.5)
- added REF**: DRILL_1.27mm, CUSTOM-FOOTPRINTS:DRILL_1.27mm, F.Cu at (153.4, 191.5)
- added REF**: DRILL_1.27mm, CUSTOM-FOOTPRINTS:DRILL_1.27mm, F.Cu at (127.6, 193.7)
- added REF**: DRILL_1.27mm, CUSTOM-FOOTPRINTS:DRILL_1.27mm, F.Cu at (200.3, 191.5)
- added REF**: Hole_2.7mm, CUSTOM-FOOTPRINTS:Hole_2.7mm, F.Cu at (133.0, 228.9)
- added REF**: DRILL_1.27mm, CUSTOM-FOOTPRINTS:DRILL_1.27mm, F.Cu at (157.8, 191.5)
- added REF**: DRILL_1.27mm, CUSTOM-FOOTPRINTS:DRILL_1.27mm, F.Cu at (179.1, 191.5)
- added REF**: DRILL_1.27mm, CUSTOM-FOOTPRINTS:DRILL_1.27mm, F.Cu at (134.3, 191.5)
- added REF**: DRILL_1.27mm, CUSTOM-FOOTPRINTS:DRILL_1.27mm, F.Cu at (198.1, 191.5)
- added REF**: DRILL_1.27mm_11.43mm, CUSTOM-FOOTPRINTS:DRILL_1.27mm_11.43mm, F.Cu at (143.8, 191.5)
- added REF**: DRILL_1.27mm, CUSTOM-FOOTPRINTS:DRILL_1.27mm, F.Cu at (80.6, 191.5)
- added REF**: DRILL_1.27mm, CUSTOM-FOOTPRINTS:DRILL_1.27mm, F.Cu at (183.5, 191.5)
- added REF**: DRILL_1.27mm, CUSTOM-FOOTPRINTS:DRILL_1.27mm, F.Cu at (174.6, 191.5)
- added REF**: DRILL_1.27mm, CUSTOM-FOOTPRINTS:DRILL_1.27mm, F.Cu at (118.7, 223.8)
- added REF**: DRILL_1.27mm_11.43mm, CUSTOM-FOOTPRINTS:DRILL_1.27mm_11.43mm, F.Cu at (167.3, 191.5)
- added REF**: DRILL_1.27mm, CUSTOM-FOOTPRINTS:DRILL_1.27mm, F.Cu at (71.8, 191.5)
- added REF**: DRILL_1.27mm, CUSTOM-FOOTPRINTS:DRILL_1.27mm, F.Cu at (230.5, 191.5)
- added REF**: DRILL_1.27mm, CUSTOM-FOOTPRINTS:DRILL_1.27mm, F.Cu at (118.7, 195.9)
- added REF**: DRILL_1.27mm, CUSTOM-FOOTPRINTS:DRILL_1.27mm, F.Cu at (136.5, 191.5)
- added REF**: DRILL_1.27mm, CUSTOM-FOOTPRINTS:DRILL_1.27mm, F.Cu at (99.7, 191.5)
- added REF**: DRILL_1.27mm_11.43mm, CUSTOM-FOOTPRINTS:DRILL_1.27mm_11.43mm, F.Cu at (261.3, 191.5)
- added REF**: DRILL_1.27mm, CUSTOM-FOOTPRINTS:DRILL_1.27mm, F.Cu at (127.6, 198.1)
- added REF**: DRILL_1.27mm, CUSTOM-FOOTPRINTS:DRILL_1.27mm, F.Cu at (223.8, 191.5)
- added REF**: DRILL_1.27mm, CUSTOM-FOOTPRINTS:DRILL_1.27mm, F.Cu at (67.3, 191.5)
- added REF**: DRILL_1.27mm, CUSTOM-FOOTPRINTS:DRILL_1.27mm, F.Cu at (118.7, 202.6)
- added REF**: DRILL_1.27mm_11.43mm, CUSTOM-FOOTPRINTS:DRILL_1.27mm_11.43mm, F.Cu at (237.8, 191.5)
- added REF**: DRILL_1.27mm, CUSTOM-FOOTPRINTS:DRILL_1.27mm, F.Cu at (76.2, 191.5)
- added REF**: DRILL_1.27mm, CUSTOM-FOOTPRINTS:DRILL_1.27mm, F.Cu at (101.9, 191.5)
- added REF**: Hole_2.7mm, CUSTOM-FOOTPRINTS:Hole_2.7mm, F.Cu at (273.4, 228.9)
- added REF**: DRILL_1.27mm, CUSTOM-FOOTPRINTS:DRILL_1.27mm, F.Cu at (155.6, 191.5)
- added REF**: DRILL_1.27mm, CUSTOM-FOOTPRINTS:DRILL_1.27mm, F.Cu at (127.6, 195.9)
- added REF**: DRILL_1.27mm, CUSTOM-FOOTPRINTS:DRILL_1.27mm, F.Cu at (275.3, 191.5)
- added REF**: DRILL_1.27mm, CUSTOM-FOOTPRINTS:DRILL_1.27mm, F.Cu at (247.3, 191.5)
- added REF**: DRILL_1.27mm_11.43mm, CUSTOM-FOOTPRINTS:DRILL_1.27mm_11.43mm, F.Cu at (87.9, 191.5)
- added REF**: DRILL_1.27mm_11.43mm, CUSTOM-FOOTPRINTS:DRILL_1.27mm_11.43mm, F.Cu at (214.3, 191.5)
- added REF**: DRILL_1.27mm, CUSTOM-FOOTPRINTS:DRILL_1.27mm, F.Cu at (127.6, 217.2)
- added REF**: DRILL_1.27mm, CUSTOM-FOOTPRINTS:DRILL_1.27mm, F.Cu at (127.6, 226.1)
- added REF**: DRILL_1.27mm, CUSTOM-FOOTPRINTS:DRILL_1.27mm, F.Cu at (127.6, 191.5)
- added REF**: DRILL_1.27mm, CUSTOM-FOOTPRINTS:DRILL_1.27mm, F.Cu at (118.7, 228.3)
- added REF**: DRILL_1.27mm, CUSTOM-FOOTPRINTS:DRILL_1.27mm, F.Cu at (118.7, 193.7)
- added REF**: DRILL_1.27mm, CUSTOM-FOOTPRINTS:DRILL_1.27mm, F.Cu at (104.1, 191.5)
- added REF**: DRILL_1.27mm, CUSTOM-FOOTPRINTS:DRILL_1.27mm, F.Cu at (151.1, 191.5)
- added REF**: DRILL_1.27mm, CUSTOM-FOOTPRINTS:DRILL_1.27mm, F.Cu at (118.7, 221.6)
- added REF**: DRILL_1.27mm, CUSTOM-FOOTPRINTS:DRILL_1.27mm, F.Cu at (176.8, 191.5)
- added REF**: DRILL_1.27mm, CUSTOM-FOOTPRINTS:DRILL_1.27mm, F.Cu at (207.0, 191.5)
- added REF**: DRILL_1.27mm, CUSTOM-FOOTPRINTS:DRILL_1.27mm, F.Cu at (127.6, 219.4)
- added REF**: DRILL_1.27mm, CUSTOM-FOOTPRINTS:DRILL_1.27mm, F.Cu at (69.5, 191.5)
- added REF**: DRILL_1.27mm, CUSTOM-FOOTPRINTS:DRILL_1.27mm, F.Cu at (121.0, 191.5)
- added REF**: DRILL_1.27mm, CUSTOM-FOOTPRINTS:DRILL_1.27mm, F.Cu at (160.0, 191.5)
- added REF**: DRILL_1.27mm, CUSTOM-FOOTPRINTS:DRILL_1.27mm, F.Cu at (181.3, 191.5)
- added REF**: DRILL_1.27mm, CUSTOM-FOOTPRINTS:DRILL_1.27mm, F.Cu at (127.6, 223.8)
- added REF**: DRILL_1.27mm, CUSTOM-FOOTPRINTS:DRILL_1.27mm, F.Cu at (127.6, 202.6)
- added REF**: DRILL_1.27mm, CUSTOM-FOOTPRINTS:DRILL_1.27mm, F.Cu at (74.0, 191.5)
- added REF**: DRILL_1.27mm_11.43mm, CUSTOM-FOOTPRINTS:DRILL_1.27mm_11.43mm, F.Cu at (111.4, 191.5)
- added REF**: DRILL_1.27mm, CUSTOM-FOOTPRINTS:DRILL_1.27mm, F.Cu at (118.7, 230.5)
- added REF**: DRILL_1.27mm_11.43mm, CUSTOM-FOOTPRINTS:DRILL_1.27mm_11.43mm, F.Cu at (127.6, 209.9)
- added REF**: DRILL_1.27mm, CUSTOM-FOOTPRINTS:DRILL_1.27mm, F.Cu at (202.6, 191.5)
- added REF**: DRILL_1.27mm, CUSTOM-FOOTPRINTS:DRILL_1.27mm, F.Cu at (273.1, 191.5)
- added REF**: DRILL_1.27mm, CUSTOM-FOOTPRINTS:DRILL_1.27mm, F.Cu at (127.6, 228.3)
- added REF**: DRILL_1.27mm, CUSTOM-FOOTPRINTS:DRILL_1.27mm, F.Cu at (249.6, 191.5)
- added REF**: DRILL_1.27mm, CUSTOM-FOOTPRINTS:DRILL_1.27mm, F.Cu at (251.8, 191.5)
- added REF**: DRILL_1.27mm, CUSTOM-FOOTPRINTS:DRILL_1.27mm, F.Cu at (132.1, 191.5)
- added REF**: DRILL_1.27mm, CUSTOM-FOOTPRINTS:DRILL_1.27mm, F.Cu at (118.7, 219.4)
- added REF**: DRILL_1.27mm, CUSTOM-FOOTPRINTS:DRILL_1.27mm, F.Cu at (97.5, 191.5)
- added REF**: DRILL_1.27mm, CUSTOM-FOOTPRINTS:DRILL_1.27mm, F.Cu at (129.9, 191.5)
- added REF**: DRILL_1.27mm, CUSTOM-FOOTPRINTS:DRILL_1.27mm, F.Cu at (127.6, 200.3)
- added REF**: DRILL_1.27mm, CUSTOM-FOOTPRINTS:DRILL_1.27mm, F.Cu at (125.4, 191.5)
- added REF**: DRILL_1.27mm, CUSTOM-FOOTPRINTS:DRILL_1.27mm, F.Cu at (228.3, 191.5)
- added U201: L7812CV, CUSTOM-FOOTPRINTS:TO-220-3_Vertical_Heatsink-SK-104_38.1mm, F.Cu at (203.2, 214.6)
- added U202: L7815CV, CUSTOM-FOOTPRINTS:TO-220-3_Vertical_Heatsink-SK-104_38.1mm, F.Cu at (161.9, 214.6)
- added U203: L7915CV, CUSTOM-FOOTPRINTS:TO-220-3_Vertical_Heatsink-SK-104_38.1mm, F.Cu at (244.5, 214.6)
- moved REF** 0.95 mm to (127.6, 178.1)
- moved REF** 0.95 mm to (127.6, 180.3)
- moved REF** 0.95 mm to (127.6, 154.6)
- moved REF** 0.95 mm to (127.6, 140.0)
- moved REF** 0.95 mm to (127.6, 109.9)
- moved REF** 0.95 mm to (127.6, 123.8)
- moved REF** 0.95 mm to (127.6, 112.1)
- moved REF** 0.95 mm to (127.6, 116.5)
- moved REF** 0.95 mm to (127.6, 114.3)
- moved REF** 0.95 mm to (127.6, 161.3)
- moved REF** 0.95 mm to (127.6, 182.6)
- moved REF** 0.95 mm to (127.6, 184.8)
- moved REF** 0.95 mm to (127.6, 189.2)
- moved REF** 0.95 mm to (127.6, 131.1)
- moved REF** 0.95 mm to (127.6, 135.6)
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- renumbered CNT101 to CNT106, CNT102 to CNT107, CNT104 to CNT108, CNT105 to CNT109, CNT106 to CNT110, CNT103 to CNT111, CNT108 to CNT112, CNT107 to CNT113
Routing:
- net PGND2: track 0.00 -> 346.3 mm
- net Net-(CNT216-Pin_4): track 0.00 -> 193.5 mm
- net Net-(CNT216-Pin_1): track 0.00 -> 183.5 mm
- net Net-(CNT214-Pin_1): track 0.00 -> 170.6 mm
- net AGND2: track 0.00 -> 157.4 mm
- net Net-(D203-+): track 0.00 -> 64.0 mm
- net Net-(CNT213-Pin_1): track 0.00 -> 48.5 mm
- net Net-(CNT213-Pin_3): track 0.00 -> 47.5 mm
- net Net-(D203--): track 0.00 -> 43.3 mm
- net Net-(CNT104-Pin_1): track 0.00 -> 36.6 mm
- net Net-(CNT103-Pin_1): track 0.00 -> 36.6 mm
- net Net-(CNT101-Pin_1): track 0.00 -> 24.4 mm
- net Net-(CNT102-Pin_1): track 0.00 -> 24.1 mm
- net Net-(CNT105-Pin_1): track 0.00 -> 18.2 mm
Other:
- board size 214.3 x 85.7 mm -> 214.3 x 128.6 mm
